File: Schematics/Command-Section/CMD_Board.kicad_pcb (KiCad board)
At the start: 2 copper layers, 280 x 186 mm, 171 parts, among them J1 USB_B, J2 Conn_02x05_Odd_Even, J3 Conn_01x04_Male, J4 Conn_02x05_Odd_Even, J5 Conn_02x05_Odd_Even, SW1 Switch_SW_DPST, SW10 Switch_SW_DPST, SW11 Switch_SW_DPST, SW12 Switch_SW_DPST, SW13 Switch_SW_DPST, SW14 Switch_SW_DPST, SW15 Switch_SW_DPST, SW16 Switch_SW_DPST, SW17 Switch_SW_DPST, SW18 Switch_SW_DPST, SW19 Switch_SW_DPST, SW2 Switch_SW_DPST, SW20 Switch_SW_DPST, SW21 Switch_SW_DPST, SW22 Switch_SW_DPST, SW23 Switch_SW_DPST, SW24 Switch_SW_DPST, SW25 Switch_SW_DPST, SW26 Switch_SW_DPST, SW27 Switch_SW_DPST, SW28 Switch_SW_DPST, SW29 Switch_SW_DPST, SW3 Switch_SW_DPST, SW30 Switch_SW_DPST, SW31 Switch_SW_DPST, SW32 Switch_SW_DPST, SW33 Switch_SW_DPST, SW34 Switch_SW_DPST, SW35 Switch_SW_DPST, SW36 Switch_SW_DPST, SW37 Switch_SW_DPST, SW38 Switch_SW_DPST, SW39 Switch_SW_DPST, SW4 Switch_SW_DPST, SW40 Switch_SW_DPST, SW41 Switch_SW_DPST, SW42 Switch_SW_DPST, SW43 Switch_SW_DPST, SW44 Switch_SW_DPST, SW45 Switch_SW_DPST, SW46 Switch_SW_DPST, SW47 Switch_SW_DPST, SW48 Switch_SW_DPST, SW49 Switch_SW_DPST, SW5 Switch_SW_DPST, SW50 Switch_SW_DPST, SW51 Switch_SW_DPST, SW52 Switch_SW_DPST, SW53 Switch_SW_DPST, SW54 Switch_SW_DPST, SW55 Switch_SW_DPST, SW56 Switch_SW_DPST, SW57 Switch_SW_DPST, SW58 Switch_SW_DPST, SW59 Switch_SW_DPST, SW6 Switch_SW_DPST, SW60 Switch_SW_DPST, SW61 Switch_SW_DPST, SW62 Switch_SW_DPST, SW63 Switch_SW_DPST, SW64 Switch_SW_DPST, SW65 Switch_SW_DPST, SW66 Switch_SW_DPST, SW67 Switch_SW_DPST, SW68 Switch_SW_DPST, SW69 Switch_SW_DPST, SW7 Switch_SW_DPST, SW8 Switch_SW_DPST, SW9 Switch_SW_DPST, U1 74HC595, U2 L7805, U3 ATmega8-16P, Y1 16MHz

Commit message: updates
Parts:
- added JP1: Jumper_2_Bridged, Jumper:SolderJumper-2_P1.3mm_Bridged_Pad1.0x1.5mm, B.Cu at (289.2, 129.8)
Connections:
- R1 pad 2: USB_INT/SER -> USB_INT
- U3 pad 11: unconnected-(U3-Pad11) -> SER_CLK
- U3 pad 25: SER_CLK -> ANALOG_3
- U3 pad 26: SER_DATA -> ANALOG_4
- U3 pad 28: unconnected-(U3-Pad28) -> SER_DATA
Routing:
- net +5V: track 8.31 -> 250.5 mm, vias 0 -> 5
- net MATRIX_8: track 496.0 -> 628.3 mm, vias 7 -> 8
- net GND: track 14.0 -> 106.0 mm, vias 0 -> 2
- net +5VA: track 120.4 -> 200.8 mm, vias 1 -> 3
- net ICSP_SCK: track 563.1 -> 640.7 mm, vias 6 -> 8
- net ANALOG_2: track 0.00 -> 77.5 mm, vias 0 -> 2
- net +12V: track 0.00 -> 63.0 mm, vias 0 -> 2
- net MATRIX_7: track 677.0 -> 738.4 mm, vias 10 -> 14
- net MATRIX_2: track 484.9 -> 543.8 mm, vias 6 -> 7
- net MATRIX_1: track 633.3 -> 689.5 mm
- net SER_CLK: track 47.1 -> 32.4 mm
- net SER_DATA: track 40.7 -> 45.0 mm
- net USB_INT: track 10.7 -> 13.0 mm
- net MATRIX_F: vias 3 -> 2
- added copper zone on B.Cu, net GND
- added copper zone on F.Cu, net GND
