File: Schematics/Command-Section/CMD_Board.kicad_sch (KiCad schematic)
At the start: 36 parts, among them J1 USB_B, J2 Conn_02x05_Odd_Even, J3 Conn_01x04_Male, J4 Conn_02x05_Odd_Even, J5 Conn_02x05_Odd_Even, U2 L7805, U3 ATmega8-16P, Y1 16MHz

Commit message: updates
Parts:
- added JP1: Jumper_2_Bridged, Jumper:SolderJumper-2_P1.3mm_Bridged_Pad1.0x1.5mm, symbol Jumper:Jumper_2_Bridged
- U1: value (none) -> 74HC595; footprint (none) -> Package_DIP:DIP-16_W7.62mm_Socket_LongPads
Connections:
- net USB_INT/SER is gone; now on net USB_INT: R1.2
- net +5V: now also JP1.1 (A)
- net +5VA: now also JP1.2 (B)
